File: End-Effector_Electronics/End-Effector_Electronics.sch (KiCad schematic (older format))
At the start: 2 parts

Commit message: Added a few components
Parts:
- added U?: BNO055, Package_LGA:LGA-28_5.2x3.8mm_P0.5mm, symbol Sensor_Motion:BNO055
- added U?: TDK_I3A4W008A033V, symbol Project_Library:TDK_I3A4W008A033V
Changed lines of the file:
@@
+	1    0    0    -1
+$EndComp
+$Comp
+L Sensor_Motion:BNO055 U?
+U 1 1 617D6C44
+P 8000 2100
+F 0 "U?" H 8000 2981 50  0000 C CNN
+F 1 "BNO055" H 8000 2890 50  0000 C CNN
+F 2 "Package_LGA:LGA-28_5.2x3.8mm_P0.5mm" H 8250 1450 50  0001 L CNN
+F 3 "https://ae-bst.resource.bosch.com/media/_tech/media/datasheets/BST_BNO055_DS000_14.pdf" H 8000 2300 50  0001 C CNN
+	1    8000 2100
+	1    0    0    -1
+$EndComp
+$Comp
+L Project_Library:TDK_I3A4W008A033V U?
+U 1 1 617D80DB
+P 7950 4300
+F 0 "U?" H 7950 4765 50  0000 C CNN
+F 1 "TDK_I3A4W008A033V" H 7950 4674 50  0000 C CNN
+F 2 "" H 7450 4600 50  0001 C CNN
+F 3 "" H 7450 4600 50  0001 C CNN
+	1    7950 4300
 	1    0    0    -1
 $EndComp

Commit message: Added libraries
libraries. Replaced BNO055
Parts:
- removed U?: BNO055, Package_LGA:LGA-28_5.2x3.8mm_P0.5mm, symbol Sensor_Motion:BNO055
- added J?: QWIIC_Generic_Conn, symbol ASTRA_Library:QWIIC_Generic_Conn
- J?: symbol SparkFun-Connectors:RASPBERRYPI-40-PIN-GPIO_SMT -> End-Effector_Electronics-rescue:RASPBERRYPI-40-PIN-GPIO_SMT-SparkFun-Connectors
Other:
- note added: "BNO055"
Changed lines of the file:
@@
 EESchema Schematic File Version 4
+LIBS:End-Effector_Electronics-cache
 EELAYER 30 0
 EELAYER END
@@
 $EndDescr
 $Comp
-L SparkFun-Connectors:RASPBERRYPI-40-PIN-GPIO_SMT J?
+L End-Effector_Electronics-rescue:RASPBERRYPI-40-PIN-GPIO_SMT-SparkFun-Connectors J?
 U 1 1 61744292
 P 1900 2750
@@
 $EndComp
 $Comp
-L Sensor_Motion:BNO055 U?
-U 1 1 617D6C44
-P 8000 2100
-F 0 "U?" H 8000 2981 50  0000 C CNN
-F 1 "BNO055" H 8000 2890 50  0000 C CNN
-F 2 "Package_LGA:LGA-28_5.2x3.8mm_P0.5mm" H 8250 1450 50  0001 L CNN
-F 3 "https://ae-bst.resource.bosch.com/media/_tech/media/datasheets/BST_BNO055_DS000_14.pdf" H 8000 2300 50  0001 C CNN
-	1    8000 2100
-	1    0    0    -1
-$EndComp
-$Comp
 L Project_Library:TDK_I3A4W008A033V U?
 U 1 1 617D80DB
@@
 	1    0    0    -1
 $EndComp
+$Comp
+L ASTRA_Library:QWIIC_Generic_Conn J?
+U 1 1 617F930F
+P 8000 1950
+F 0 "J?" H 8178 1696 50  0000 L CNN
+F 1 "QWIIC_Generic_Conn" H 8178 1605 50  0000 L CNN
+F 2 "" H 8000 1950 50  0001 C CNN
+F 3 "" H 8000 1950 50  0001 C CNN
+	1    8000 1950
+	1    0    0    -1
+$EndComp
+Text Notes 7800 1850 0    50   ~ 0
+BNO055
 $EndSCHEMATC

Commit message: added sheet for 5v supply
Parts:
- J?: symbol End-Effector_Electronics-rescue:RASPBERRYPI-40-PIN-GPIO_SMT-SparkFun-Connectors -> End-Effector_Electronics-rescue:RASPBERRYPI-40-PIN-GPIO_SMT-SparkFun-Connectors-End-Effector_Electronics-rescue
Changed lines of the file:
@@
 EESchema Schematic File Version 4
-LIBS:End-Effector_Electronics-cache
 EELAYER 30 0
 EELAYER END
 $Descr A4 11693 8268
 encoding utf-8
-Sheet 1 1
+Sheet 1 2
 Title ""
 Date ""
@@
 $EndDescr
 $Comp
-L End-Effector_Electronics-rescue:RASPBERRYPI-40-PIN-GPIO_SMT-SparkFun-Connectors J?
+L End-Effector_Electronics-rescue:RASPBERRYPI-40-PIN-GPIO_SMT-SparkFun-Connectors-End-Effector_Electronics-rescue J?
 U 1 1 61744292
 P 1900 2750
@@
 Text Notes 7800 1850 0    50   ~ 0
 BNO055
+$Sheet
+S 4900 4050 800  750
+U 617D965B
+F0 "5V Supply" 50
+F1 "5v_Supply.sch" 50
+F2 "Vin-" I L 4900 4600 50
+F3 "Vin+" I L 4900 4250 50
+F4 "Vout-" O R 5700 4600 50
+F5 "Vout+" O R 5700 4250 50
+$EndSheet
 $EndSCHEMATC

Commit message: 12v supply
and bno
Parts:
- added C?: 0.1u, symbol Device:C_Small
- added C?: 22uF, symbol Device:CP1_Small
- added C?: 33u, symbol Device:CP1_Small
- added Q?: Q_NMOS_GSD, symbol Device:Q_NMOS_GSD
- added R?: 1.82k, symbol Device:R_Small
- added R?: 100k, symbol Device:R_Small
- J?: symbol End-Effector_Electronics-rescue:RASPBERRYPI-40-PIN-GPIO_SMT-SparkFun-Connectors-End-Effector_Electronics-rescue -> End-Effector_Electronics-rescue:RASPBERRYPI-40-PIN-GPIO_SMT-SparkFun-Connectors-End-Effector_Electronics-rescue-End-Eff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
Connections:
- net labels added: +12V, +3.3V, +BATT, 12V_Disable, GND, SCL, SDA
- wire segments 0 -> 34
Changed lines of the file:
@@
 EESchema Schematic File Version 4
+LIBS:End-Effector_Electronics-cache
 EELAYER 30 0
 EELAYER END
@@
 $EndDescr
 $Comp
-L End-Effector_Electronics-rescue:RASPBERRYPI-40-PIN-GPIO_SMT-SparkFun-Connectors-End-Effector_Electronics-rescue J?
+L End-Effector_Electronics-rescue:RASPBERRYPI-40-PIN-GPIO_SMT-SparkFun-Connectors-End-Effector_Electronics-rescue-End-Effector_Electronics-rescue J?
 U 1 1 61744292
 P 1900 2750
@@
 F5 "Vout+" O R 5700 4250 50
 $EndSheet
+$Comp
+L Device:R_Small R?
+U 1 1 617D861F
+P 8700 4400
+F 0 "R?" H 8759 4446 50  0000 L CNN
+F 1 "1.82k" H 8759 4355 50  0000 L CNN
+F 2 "" H 8700 4400 50  0001 C CNN
+F 3 "~" H 8700 4400 50  0001 C CNN
+	1    8700 4400
+	1    0    0    -1
+$EndComp
+Wire Wire Line
+	8700 4300 8450 4300
+Wire Wire Line
+	8700 4500 8450 4500
+$Comp
+L Device:C_Small C?
+U 1 1 617D8F46
+P 9000 4250
+F 0 "C?" H 9092 4296 50  0000 L CNN
+F 1 "0.1u" H 9092 4205 50  0000 L CNN
+F 2 "" H 9000 4250 50  0001 C CNN
+F 3 "~" H 9000 4250 50  0001 C CNN
+	1    9000 4250
+	1    0    0    -1
+$EndComp
+$Comp
+L Device:CP1_Small C?
+U 1 1 617D9903
+P 9300 4250
+F 0 "C?" H 9391 4296 50  0000 L CNN
+F 1 "22uF" H 9391 4205 50  0000 L CNN
+F 2 "" H 9300 4250 50  0001 C CNN
+F 3 "~" H 9300 4250 50  0001 C CNN
+	1    9300 4250
+	1    0    0    -1
+$EndComp
+Wire Wire Line
+	9000 4150 9000 4100
+Wire Wire Line
+	9000 4100 8450 4100
+Wire Wire Line
+	9300 4150 9300 4100
+Wire Wire Line
+	9300 4100 9000 4100
+Connection ~ 9000 4100
+Wire Wire Line
+	9300 4350 9300 4500
+Wire Wire Line
+	9300 4500 9000 4500
+Connection ~ 8700 4500
+Wire Wire Line
+	9000 4350 9000 4500
+Connection ~ 9000 4500
+Wire Wire Line
+	9000 4500 8700 4500
+Wire Wire Line
+	9000 4600 9000 4500
+$Comp
+L power:GND #PWR?
+U 1 1 617DEA0F
+P 9000 4600
+F 0 "#PWR?" H 9000 4350 50  0001 C CNN
+F 1 "GND" H 9005 4427 50  0000 C CNN
+F 2 "" H 9000 4600 50  0001 C CNN
+F 3 "" H 9000 4600 50  0001 C CNN
+	1    9000 4600
+	1    0    0    -1
+$EndComp
+$Comp
+L power:+12V #PWR?
+U 1 1 617DEE5D
+P 9350 4050
+F 0 "#PWR?" H 9350 3900 50  0001 C CNN
+F 1 "+12V" H 9365 4223 50  0000 C CNN
+F 2 "" H 9350 4050 50  0001 C CNN
+F 3 "" H 9350 4050 50  0001 C CNN
+	1    9350 4050
+	1    0    0    -1
+$EndComp
+Wire Wire Line
+	9350 4050 9350 4100
+Wire Wire Line
+	9350 4100 9300 4100
+Connection ~ 9300 4100
+$Comp
+L power:+BATT #PWR?
+U 1 1 617DFAEB
+P 7300 3950
+F 0 "#PWR?" H 7300 3800 50  0001 C CNN
+F 1 "+BATT" H 7315 4123 50  0000 C CNN
+F 2 "" H 7300 3950 50  0001 C CNN
+F 3 "" H 7300 3950 50  0001 C CNN
+	1    7300 3950
+	1    0    0    -1
+$EndComp
+$Comp
+L Device:CP1_Small C?
+U 1 1 617E08C5
+P 7100 4100
+F 0 "C?" V 6872 4100 50  0000 C CNN
+F 1 "33u" V 6963 4100 50  0000 C CNN
+F 2 "" H 7100 4100 50  0001 C CNN
+F 3 "~" H 7100 4100 50  0001 C CNN
+	1    7100 4100
+	0    1    1    0
+$EndComp
+Wire Wire Line
+	7450 4100 7300 4100
+Wire Wire Line
+	7300 3950 7300 4100
+Connection ~ 7300 4100
+Wire Wire Line
+	7300 4100 7200 4100
+Wire Wire Line
+	7000 4100 6900 4100
+Wire Wire Line
+	6900 4100 6900 4150
+$Comp
+L Device:Q_NMOS_GSD Q?
+U 1 1 617E24A7
+P 6600 4600
+F 0 "Q?" H 6806 4646 50  0000 L CNN
+F 1 "Q_NMOS_GSD" H 6806 4555 50  0000 L CNN
+F 2 "" H 6800 4700 50  0001 C CNN
+F 3 "~" H 6600 4600 50  0001 C CNN
+	1    6600 4600
+	1    0    0    -1
+$EndComp
+Wire Wire Line
+	7450 4300 6700 4300
+Wire Wire Line
+	6700 4300 6700 4400
+$Comp
+L power:GND #PWR?
+U 1 1 617E1587
+P 6900 4150
+F 0 "#PWR?" H 6900 3900 50  0001 C CNN
+F 1 "GND" H 6800 4050 50  0000 C CNN
+F 2 "" H 6900 4150 50  0001 C CNN
+F 3 "" H 6900 4150 50  0001 C CNN
+	1    6900 4150
+	1    0    0    -1
+$EndComp
+$Comp
+L Device:R_Small R?
+U 1 1 617E5A4B
+P 6350 4800
+F 0 "R?" H 6409 4846 50  0000 L CNN
+F 1 "100k" H 6409 4755 50  0000 L CNN
+F 2 "" H 6350 4800 50  0001 C CNN
+F 3 "~" H 6350 4800 50  0001 C CNN
+	1    6350 4800
+	1    0    0    -1
+$EndComp
+$Comp
+L power:GND #PWR?
+U 1 1 617E70E3
+P 6700 4950
+F 0 "#PWR?" H 6700 4700 50  0001 C CNN
+F 1 "GND" H 6705 4777 50  0000 C CNN
+F 2 "" H 6700 4950 50  0001 C CNN
+F 3 "" H 6700 4950 50  0001 C CNN
+	1    6700 4950
+	1    0    0    -1
+$EndComp
+Wire Wire Line
+	6400 4600 6350 4600
+Wire Wire Line
+	6350 4600 6350 4700
+Wire Wire Line
+	6350 4900 6700 4900
+Wire Wire Line
+	6700 4900 6700 4950
+Wire Wire Line
+	6700 4800 6700 4900
+Connection ~ 6700 4900
+Wire Wire Line
+	6350 4600 6300 4600
+Connection ~ 6350 4600
+Text Label 6300 4600 2    50   ~ 0
+12V_Disable
+Wire Wire Line
+	7750 2100 7450 2100
+Wire Wire Line
+	7750 2200 7450 2200
+Wire Wire Line
+	2500 1650 2700 1650
+Wire Wire Line
+	2500 1750 2700 1750
+Text Label 2700 1650 0    50   ~ 0
+SDA
+Text Label 2700 1750 0    50   ~ 0
+SCL
+Text Label 7450 2100 2    50   ~ 0
+SCL
+Text Label 7450 2200 2    50   ~ 0
+SDA
+$Comp
+L power:+3.3V #PWR?
+U 1 1 617EBD30
+P 7150 2250
+F 0 "#PWR?" H 7150 2100 50  0001 C CNN
+F 1 "+3.3V" H 7165 2423 50  0000 C CNN
+F 2 "" H 7150 2250 50  0001 C CNN
+F 3 "" H 7150 2250 50  0001 C CNN
+	1    7150 2250
+	1    0    0    -1
+$EndComp
+$Comp
+L power:GND #PWR?
+U 1 1 617EC57E
+P 7600 2500
+F 0 "#PWR?" H 7600 2250 50  0001 C CNN
+F 1 "GND" H 7605 2327 50  0000 C CNN
+F 2 "" H 7600 2500 50  0001 C CNN
+F 3 "" H 7600 2500 50  0001 C CNN
+	1    7600 2500
+	1    0    0    -1
+$EndComp
+Wire Wire Line
+	7750 2400 7600 2400
+Wire Wire Line
+	7600 2400 7600 2500
+Wire Wire Line
+	7750 2300 7150 2300
+Wire Wire Line
+	7150 2300 7150 2250
 $EndSCHEMATC

Commit message: Fixed broken thingy
Parts:
- removed J?: RASPBERRYPI-40-PIN-GPIO_SMT, 2X20_SHROUDED_SMT, symbol End-Effector_Electronics-rescue:RASPBERRYPI-40-PIN-GPIO_SMT-SparkFun-Connectors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
- added J?: Raspberry_Pi_2_3, symbol Connector:Raspberry_Pi_2_3
Changed lines of the file:
@@
 EESchema Schematic File Version 4
-LIBS:End-Effector_Electronics-cache
 EELAYER 30 0
 EELAYER END
@@
 $EndDescr
 $Comp
-L End-Effector_Electronics-rescue:RASPBERRYPI-40-PIN-GPIO_SMT-SparkFun-Connectors-End-Effector_Electronics-rescue-End-Effector_Electronics-rescue J?
-U 1 1 61744292
-P 1900 2750
-F 0 "J?" H 1900 4210 45  0000 C CNN
-F 1 "RASPBERRYPI-40-PIN-GPIO_SMT" H 1900 4126 45  0000 C CNN
-F 2 "2X20_SHROUDED_SMT" H 1900 4050 20  0001 C CNN
-F 3 "" H 1900 2750 50  0001 C CNN
-F 4 "CONN-13143" H 1900 4031 60  0000 C CNN "Field4"
-	1    1900 2750
-	1    0    0    -1
-$EndComp
-$Comp
 L Project_Library:LynxServo J?
 U 1 1 61745589
@@
 	7750 2200 7450 2200
 Wire Wire Line
-	2500 1650 2700 1650
-Wire Wire Line
-	2500 1750 2700 1750
-Text Label 2700 1650 0    50   ~ 0
+	2950 2000 3150 2000
+Wire Wire Line
+	2950 2100 3150 2100
+Text Label 3150 2000 0    50   ~ 0
 SDA
-Text Label 2700 1750 0    50   ~ 0
+Text Label 3150 2100 0    50   ~ 0
 SCL
 Text Label 7450 2100 2    50   ~ 0
@@
 Wire Wire Line
 	7150 2300 7150 2250
+$Comp
+L Connector:Raspberry_Pi_2_3 J?
+U 1 1 617E71E0
+P 2150 2600
+F 0 "J?" H 2150 4081 50  0000 C CNN
+F 1 "Raspberry_Pi_2_3" H 2150 3990 50  0000 C CNN
+F 2 "" H 2150 2600 50  0001 C CNN
+F 3 "https://www.raspberrypi.org/documentation/hardware/raspberrypi/schematics/rpi_SCH_3bplus_1p0_reduced.pdf" H 2150 2600 50  0001 C CNN
+	1    2150 2600
+	1    0    0    -1
+$EndComp
 $EndSCHEMATC

Commit message: Added some stuff
very description
Parts:
- added BT?: XT60_Battery_Connector, symbol ASTRA_Library:XT60_Battery_Connector
Connections:
- net +12V: now also J?.2 (Vcc)
- net +3V3: now also J?.1 (3V3), J?.17 (3V3)
- net +BATT: now also BT?.2 (Pos)
- net GND: now also J?.14 (GND), J?.20 (GND), J?.25 (GND), J?.3 (GND), J?.30 (GND), J?.34 (GND), J?.39 (GND), J?.6 (GND), J?.9 (GND), BT?.1 (Neg)
- net ServoRX: now reaches J?.1 (ServoRX)
- net ServoRX: now also J?.8 (GPIO14/TXD)
- net ServoTX: now reaches J?.4 (ServoTX)
- net ServoTX: now also J?.10 (GPIO15/RXD)
- net +5V: now reaches J?.2 (5V)
- net +5V: now also J?.4 (5V)
Changed lines of the file:
@@
 BNO055
 $Sheet
-S 4900 4050 800  750
+S 4300 3950 800  750
 U 617D965B
 F0 "5V Supply" 50
 F1 "5v_Supply.sch" 50
-F2 "Vin-" I L 4900 4600 50
-F3 "Vin+" I L 4900 4250 50
-F4 "Vout-" O R 5700 4600 50
-F5 "Vout+" O R 5700 4250 50
+F2 "Vin-" I L 4300 4500 50
+F3 "Vin+" I L 4300 4150 50
+F4 "Vout-" O R 5100 4500 50
+F5 "Vout+" O R 5100 4150 50
 $EndSheet
 $Comp
@@
 U 1 1 617E71E0
 P 2150 2600
-F 0 "J?" H 2150 4081 50  0000 C CNN
-F 1 "Raspberry_Pi_2_3" H 2150 3990 50  0000 C CNN
+F 0 "J?" H 2500 3950 50  0000 C CNN
+F 1 "Raspberry_Pi_2_3" H 2800 3850 50  0000 C CNN
 F 2 "" H 2150 2600 50  0001 C CNN
 F 3 "https://www.raspberrypi.org/documentation/hardware/raspberrypi/schematics/rpi_SCH_3bplus_1p0_reduced.pdf" H 2150 2600 50  0001 C CNN
@@
 	1    0    0    -1
 $EndComp
+$Comp
+L ASTRA_Library:XT60_Battery_Connector BT?
+U 1 1 617EE7FC
+P 3300 5050
+F 0 "BT?" H 3428 5096 50  0000 L CNN
+F 1 "XT60_Battery_Connector" H 3428 5005 50  0000 L CNN
+F 2 "" H 3300 5050 50  0001 C CNN
+F 3 "" H 3300 5050 50  0001 C CNN
+	1    3300 5050
+	1    0    0    -1
+$EndComp
+$Comp
+L power:+BATT #PWR?
+U 1 1 617EF1D8
+P 3300 4800
+F 0 "#PWR?" H 3300 4650 50  0001 C CNN
+F 1 "+BATT" H 3315 4973 50  0000 C CNN
+F 2 "" H 3300 4800 50  0001 C CNN
+F 3 "" H 3300 4800 50  0001 C CNN
+	1    3300 4800
+	1    0    0    -1
+$EndComp
+$Comp
+L power:GND #PWR?
+U 1 1 617EF57A
+P 3300 5300
+F 0 "#PWR?" H 3300 5050 50  0001 C CNN
+F 1 "GND" H 3305 5127 50  0000 C CNN
+F 2 "" H 3300 5300 50  0001 C CNN
+F 3 "" H 3300 5300 50  0001 C CNN
+	1    3300 5300
+	1    0    0    -1
+$EndComp
+$Comp
+L power:+BATT #PWR?
+U 1 1 617EF8D6
+P 4050 4150
+F 0 "#PWR?" H 4050 4000 50  0001 C CNN
+F 1 "+BATT" H 4065 4323 50  0000 C CNN
+F 2 "" H 4050 4150 50  0001 C CNN
+F 3 "" H 4050 4150 50  0001 C CNN
+	1    4050 4150
+	1    0    0    -1
+$EndComp
+Wire Wire Line
+	4300 4150 4050 4150
+$Comp
+L power:GND #PWR?
+U 1 1 617F04C2
+P 4050 4500
+F 0 "#PWR?" H 4050 4250 50  0001 C CNN
+F 1 "GND" H 4055 4327 50  0000 C CNN
+F 2 "" H 4050 4500 50  0001 C CNN
+F 3 "" H 4050 4500 50  0001 C CNN
+	1    4050 4500
+	1    0    0    -1
+$EndComp
+Wire Wire Line
+	4050 4500 4300 4500
+$Comp
+L power:+12V #PWR?
+U 1 1 617F1DE8
+P 3900 1750
+F 0 "#PWR?" H 3900 1600 50  0001 C CNN
+F 1 "+12V" H 3915 1923 50  0000 C CNN
+F 2 "" H 3900 1750 50  0001 C CNN
+F 3 "" H 3900 1750 50  0001 C CNN
+	1    3900 1750
+	1    0    0    -1
+$EndComp
+Wire Wire Line
+	4400 1750 3900 1750
+$Comp
+L power:GND #PWR?
+U 1 1 617F2B7C
+P 3900 1850
+F 0 "#PWR?" H 3900 1600 50  0001 C CNN
+F 1 "GND" H 3905 1677 50  0000 C CNN
+F 2 "" H 3900 1850 50  0001 C CNN
+F 3 "" H 3900 1850 50  0001 C CNN
+	1    3900 1850
+	1    0    0    -1
+$EndComp
+Wire Wire Line
+	3900 1850 4400 1850
+$Comp
+L power:+5V #PWR?
+U 1 1 617F3BF6
+P 5350 4150
+F 0 "#PWR?" H 5350 4000 50  0001 C CNN
+F 1 "+5V" H 5365 4323 50  0000 C CNN
+F 2 "" H 5350 4150 50  0001 C CNN
+F 3 "" H 5350 4150 50  0001 C CNN
+	1    5350 4150
+	1    0    0    -1
+$EndComp
+Wire Wire Line
+	5350 4150 5100 4150
+$Comp
+L power:GND #PWR?
+U 1 1 617F487C
+P 5350 4500
+F 0 "#PWR?" H 5350 4250 50  0001 C CNN
+F 1 "GND" H 5355 4327 50  0000 C CNN
+F 2 "" H 5350 4500 50  0001 C CNN
+F 3 "" H 5350 4500 50  0001 C CNN
+	1    5350 4500
+	1    0    0    -1
+$EndComp
+Wire Wire Line
+	5350 4500 5100 4500
+$Comp
+L power:+5V #PWR?
+U 1 1 617F6C42
+P 2000 1150
+F 0 "#PWR?" H 2000 1000 50  0001 C CNN
+F 1 "+5V" H 2015 1323 50  0000 C CNN
+F 2 "" H 2000 1150 50  0001 C CNN
+F 3 "" H 2000 1150 50  0001 C CNN
+	1    2000 1150
+	1    0    0    -1
+$EndComp
+Wire Wire Line
+	2000 1150 2050 1150
+Wire Wire Line
+	2050 1150 2050 1300
+Wire Wire Line
+	2000 1150 1950 1150
+Wire Wire Line
+	1950 1150 1950 1300
+Connection ~ 2000 1150
+$Comp
+L power:+3.3V #PWR?
+U 1 1 617F96F6
+P 2300 1150
+F 0 "#PWR?" H 2300 1000 50  0001 C CNN
+F 1 "+3.3V" H 2315 1323 50  0000 C CNN
+F 2 "" H 2300 1150 50  0001 C CNN
+F 3 "" H 2300 1150 50  0001 C CNN
+	1    2300 1150
+	1    0    0    -1
+$EndComp
+Wire Wire Line
+	2350 1300 2350 1150
+Wire Wire Line
+	2350 1150 2300 1150
+Wire Wire Line
+	2300 1150 2250 1150
+Wire Wire Line
+	2250 1150 2250 1300
+Connection ~ 2300 1150
+$Comp
+L power:GND #PWR?
+U 1 1 617FBBC2
+P 2100 4100
+F 0 "#PWR?" H 2100 3850 50  0001 C CNN
+F 1 "GND" H 2105 3927 50  0000 C CNN
+F 2 "" H 2100 4100 50  0001 C CNN
+F 3 "" H 2100 4100 50  0001 C CNN
+	1    2100 4100
+	1    0    0    -1
+$EndComp
+Wire Wire Line
+	2100 4100 2100 3900
+Wire Wire Line
+	2100 3900 2050 3900
+Connection ~ 1850 3900
+Wire Wire Line
+	1850 3900 1750 3900
+Connection ~ 1950 3900
+Wire Wire Line
+	1950 3900 1850 3900
+Connection ~ 2050 3900
+Wire Wire Line
+	2050 3900 1950 3900
+Wire Wire Line
+	2450 3900 2350 3900
+Connection ~ 2100 3900
+Connection ~ 2150 3900
+Wire Wire Line
+	2150 3900 2100 3900
+Connection ~ 2250 3900
+Wire Wire Line
+	2250 3900 2150 3900
+Connection ~ 2350 3900
+Wire Wire Line
+	2350 3900 2250 3900
+Wire Wire Line
+	4400 1650 4350 1650
+Wire Wire Line
+	4400 1950 4350 1950
+Text Label 4350 1650 2    50   ~ 0
+ServoRX
+Text Label 4350 1950 2    50   ~ 0
+ServoTX
+Text Label 1150 1700 2    50   ~ 0
+ServoRX
+Wire Wire Line
+	1150 1700 1350 1700
+Wire Wire Line
+	1350 1800 1150 1800
+Text Label 1150 1800 2    50   ~ 0
+ServoTX
 $EndSCHEMATC

Commit message: Forgot to commit latest changes
Parts:
- added Q2: DMMT3906, symbol Project_Library:DMMT3906
- added Q?: Q_PMOS_GSD, symbol Device:Q_PMOS_GSD
- added R?: DNP, symbol Device:R_Small
- added R? (x2): 10k, symbol Device:R_Small
- added R?: 47k, symbol Device:R_Small
- added U2: CAT24C32, symbol Project_Library:CAT24C32
- gave numbers to parts that had none: 11
Connections:
- net +3V3: now also R?.2, U2.8 (VCC)
- net +5V: now also Q2.1 (E1), Q?.3 (D); no longer J1.2 (5V), J1.4 (5V)
- net GND: now also R?.1, R?.2, R?.2, U2.1 (A0), U2.2 (A1), U2.3 (A2), U2.4 (GND)
- net ID_SDA: now reaches J1.27 (ID_SD/GPIO0)
- net ID_SDA: now also U2.5 (SDA)
- net ID_SCL: now reaches J1.28 (ID_SC/GPIO1)
- net ID_SCL: now also U2.6 (SCL)
- new net: R?.1, R?.1, U2.7 (WP)
- new net: Q2.4 (C2), Q?.1 (G), R?.1
- new net: Q2.5 (B12), Q2.6 (C1), R?.2
- new net 5V_RPI: J1.2 (5V), J1.4 (5V), Q2.3 (E2), Q?.2 (S)
Other:
- moved on the sheet: BT1
