File: End-Effector_Electronics/End-Effector_Electronics.sch (KiCad schematic (older format))
At the start: 18 parts, among them J1 Raspberry_Pi_2_3, J2 LynxServo, J3 QWIIC_Generic_Conn, Q2 DMMT3906, Q3 Q_NMOS_GSD, U2 CAT24C32, U3 TDK_I3A4W008A033V

Commit message: Started associating components
Parts:
- added H1, H2, H3, H4: MountingHole_Pad, symbol Mechanical:MountingHole_Pad
- added J4: LynxServo, Connector_Molex:Molex_SPOX_5268-04A_1x04_P2.50mm_Horizontal, symbol Project_Library:LynxServo
- BT1: value XT60_Battery_Connector -> XT_Battery_Connector
- C6: Digikey Part Num (none) -> n/a
- R3, R4, R5: renamed from R?; Digikey Part Num (none) -> n/a
- gave numbers to parts that had none: 2
Connections:
- net +12V: now also J4.2 (Vcc)
- net 5V_RPI: no longer J1.2 (5V), J1.4 (5V)
- net GND: now also J4.3 (GND)
- net ServoRX: now also J4.1 (ServoRX)
- net ServoTX: now also J4.4 (ServoTX)
Changed lines of the file:
@@
 F 2 "" H 9000 4250 50  0001 C CNN
 F 3 "~" H 9000 4250 50  0001 C CNN
+F 4 "n/a" H 9000 4250 50  0001 C CNN "Digikey Part Num"
 	1    9000 4250
 	1    0    0    -1
@@
 P 1250 6850
 F 0 "BT1" H 1378 6896 50  0000 L CNN
-F 1 "XT60_Battery_Connector" H 1378 6805 50  0000 L CNN
+F 1 "XT_Battery_Connector" H 1378 6805 50  0000 L CNN
 F 2 "" H 1250 6850 50  0001 C CNN
 F 3 "" H 1250 6850 50  0001 C CNN
@@
 	1    0    0    -1
 $EndComp
-Wire Wire Line
-	2050 1150 2050 1300
-Wire Wire Line
-	1950 1150 1950 1300
 $Comp
 L power:+3.3V #PWR03
@@
 	2850 6800 2850 7000
 $Comp
-L power:GND #PWR?
+L power:GND #PWR019
 U 1 1 61828A76
 P 3050 7000
-F 0 "#PWR?" H 3050 6750 50  0001 C CNN
+F 0 "#PWR019" H 3050 6750 50  0001 C CNN
 F 1 "GND" H 3055 6827 50  0000 C CNN
 F 2 "" H 3050 7000 50  0001 C CNN
@@
 	3050 7000 3250 7000
 $Comp
-L Device:R_Small R?
+L Device:R_Small R3
 U 1 1 61829043
 P 3700 7150
-F 0 "R?" H 3759 7196 50  0000 L CNN
+F 0 "R3" H 3759 7196 50  0000 L CNN
 F 1 "DNP" H 3759 7105 50  0000 L CNN
 F 2 "" H 3700 7150 50  0001 C CNN
 F 3 "~" H 3700 7150 50  0001 C CNN
+F 4 "n/a" H 3700 7150 50  0001 C CNN "Digikey Part Num"
 	1    3700 7150
 	1    0    0    -1
 $EndComp
 $Comp
-L Device:R_Small R?
+L Device:R_Small R4
 U 1 1 61829E44
 P 3950 6800
-F 0 "R?" V 3846 6800 50  0000 C CNN
+F 0 "R4" V 3846 6800 50  0000 C CNN
 F 1 "10k" V 3755 6800 50  0000 C CNN
 F 2 "" H 3950 6800 50  0001 C CNN
 F 3 "~" H 3950 6800 50  0001 C CNN
+F 4 "n/a" H 3950 6800 50  0001 C CNN "Digikey Part Num"
 	1    3950 6800
 	0    -1   -1   0
@@
 Connection ~ 3700 6800
 $Comp
-L power:+3.3V #PWR?
+L power:+3.3V #PWR022
 U 1 1 61830169
 P 4300 6800
-F 0 "#PWR?" H 4300 6650 50  0001 C CNN
+F 0 "#PWR022" H 4300 6650 50  0001 C CNN
 F 1 "+3.3V" H 4315 6973 50  0000 C CNN
 F 2 "" H 4300 6800 50  0001 C CNN
@@
 	4300 6800 4050 6800
 $Comp
-L power:GND #PWR?
+L power:GND #PWR021
 U 1 1 61832C44
 P 3700 7350
-F 0 "#PWR?" H 3700 7100 50  0001 C CNN
+F 0 "#PWR021" H 3700 7100 50  0001 C CNN
 F 1 "GND" H 3705 7177 50  0000 C CNN
 F 2 "" H 3700 7350 50  0001 C CNN
@@
 	3700 7350 3700 7250
 $Comp
-L power:+3.3V #PWR?
+L power:+3.3V #PWR020
 U 1 1 618355B6
 P 3250 6400
-F 0 "#PWR?" H 3250 6250 50  0001 C CNN
+F 0 "#PWR020" H 3250 6250 50  0001 C CNN
 F 1 "+3.3V" H 3265 6573 50  0000 C CNN
 F 2 "" H 3250 6400 50  0001 C CNN
@@
 	1    0    0    -1
 $EndComp
-Text Label 2000 1150 1    50   ~ 0
-5V_RPI
 Text Label 6100 6100 0    50   ~ 0
 5V_RPI
@@
 	4700 6100 5200 6100
 Wire Wire Line
-	1950 1150 2050 1150
-Wire Wire Line
 	5600 6100 6100 6100
 $Comp
-L Device:R_Small R?
+L Device:R_Small R5
 U 1 1 6183BBC3
 P 5200 7200
-F 0 "R?" H 5141 7154 50  0000 R CNN
+F 0 "R5" H 5141 7154 50  0000 R CNN
 F 1 "10k" H 5141 7245 50  0000 R CNN
 F 2 "" H 5200 7200 50  0001 C CNN
 F 3 "~" H 5200 7200 50  0001 C CNN
+F 4 "n/a" H 5200 7200 50  0001 C CNN "Digikey Part Num"
 	1    5200 7200
 	1    0    0    1
 $EndComp
 $Comp
-L Device:R_Small R?
+L Device:R_Small R6
 U 1 1 6183BFF4
 P 5600 7200
-F 0 "R?" H 5659 7246 50  0000 L CNN
+F 0 "R6" H 5659 7246 50  0000 L CNN
 F 1 "47k" H 5659 7155 50  0000 L CNN
 F 2 "" H 5600 7200 50  0001 C CNN
@@
 $EndComp
 $Comp
-L power:GND #PWR?
+L power:GND #PWR023
 U 1 1 6183CD37
 P 5200 7300
-F 0 "#PWR?" H 5200 7050 50  0001 C CNN
+F 0 "#PWR023" H 5200 7050 50  0001 C CNN
 F 1 "GND" H 5205 7127 50  0000 C CNN
 F 2 "" H 5200 7300 50  0001 C CNN
@@
 $EndComp
 $Comp
-L power:GND #PWR?
+L power:GND #PWR024
 U 1 1 6183D0C2
 P 5600 7300
-F 0 "#PWR?" H 5600 7050 50  0001 C CNN
+F 0 "#PWR024" H 5600 7050 50  0001 C CNN
 F 1 "GND" H 5605 7127 50  0000 C CNN
 F 2 "" H 5600 7300 50  0001 C CNN
@@
 Connection ~ 5200 6100
 $Comp
-L Device:Q_PMOS_GSD Q?
+L Device:Q_PMOS_GSD Q1
 U 1 1 618633DB
 P 5400 6200
-F 0 "Q?" V 5742 6200 50  0000 C CNN
+F 0 "Q1" V 5742 6200 50  0000 C CNN
 F 1 "Q_PMOS_GSD" V 5651 6200 50  0000 C CNN
 F 2 "" H 5600 6300 50  0001 C CNN
@@
 	0    -1   -1   0
 $EndComp
+$Comp
+L Project_Library:LynxServo J4
+U 1 1 61903138
+P 4700 2650
+F 0 "J4" H 4928 2696 50  0000 L CNN
+F 1 "LynxServo" H 4928 2605 50  0000 L CNN
+F 2 "Connector_Molex:Molex_SPOX_5268-04A_1x04_P2.50mm_Horizontal" H 4700 2950 50  0001 C CNN
+F 3 "" H 4700 2950 50  0001 C CNN
+F 4 "23-0022057045-ND" H 4700 2950 50  0001 C CNN "Digikey Part Num"
+	1    4700 2650
+	1    0    0    -1
+$EndComp
+$Comp
+L power:+12V #PWR025
+U 1 1 619034EA
+P 3900 2600
+F 0 "#PWR025" H 3900 2450 50  0001 C CNN
+F 1 "+12V" H 3915 2773 50  0000 C CNN
+F 2 "" H 3900 2600 50  0001 C CNN
+F 3 "" H 3900 2600 50  0001 C CNN
+	1    3900 2600
+	1    0    0    -1
+$EndComp
+Wire Wire Line
+	4400 2600 3900 2600
+$Comp
+L power:GND #PWR026
+U 1 1 619034F5
+P 3900 2700
+F 0 "#PWR026" H 3900 2450 50  0001 C CNN
+F 1 "GND" H 3905 2527 50  0000 C CNN
+F 2 "" H 3900 2700 50  0001 C CNN
+F 3 "" H 3900 2700 50  0001 C CNN
+	1    3900 2700
+	1    0    0    -1
+$EndComp
+Wire Wire Line
+	3900 2700 4400 2700
+Wire Wire Line
+	4400 2500 4350 2500
+Wire Wire Line
+	4400 2800 4350 2800
+Text Label 4350 2500 2    50   ~ 0
+ServoRX
+Text Label 4350 2800 2    50   ~ 0
+ServoTX
+$Comp
+L Mechanical:MountingHole_Pad H1
+U 1 1 6190ADE3
+P 10000 950
+F 0 "H1" V 9954 1100 50  0000 L CNN
+F 1 "MountingHole_Pad" V 10045 1100 50  0000 L CNN
+F 2 "" H 10000 950 50  0001 C CNN
+F 3 "~" H 10000 950 50  0001 C CNN
+	1    10000 950
+	0    1    1    0
+$EndComp
+$Comp
+L Mechanical:MountingHole_Pad H2
+U 1 1 6190BC15
+P 10000 1100
+F 0 "H2" V 9954 1250 50  0000 L CNN
+F 1 "MountingHole_Pad" V 10045 1250 50  0000 L CNN
+F 2 "" H 10000 1100 50  0001 C CNN
+F 3 "~" H 10000 1100 50  0001 C CNN
+	1    10000 1100
+	0    1    1    0
+$EndComp
+$Comp
+L Mechanical:MountingHole_Pad H3
+U 1 1 6190BDDC
+P 10000 1250
+F 0 "H3" V 9954 1400 50  0000 L CNN
+F 1 "MountingHole_Pad" V 10045 1400 50  0000 L CNN
+F 2 "" H 10000 1250 50  0001 C CNN
+F 3 "~" H 10000 1250 50  0001 C CNN
+	1    10000 1250
+	0    1    1    0
+$EndComp
+$Comp
+L Mechanical:MountingHole_Pad H4
+U 1 1 6190BF74
+P 10000 1400
+F 0 "H4" V 9954 1550 50  0000 L CNN
+F 1 "MountingHole_Pad" V 10045 1550 50  0000 L CNN
+F 2 "" H 10000 1400 50  0001 C CNN
+F 3 "~" H 10000 1400 50  0001 C CNN
+	1    10000 1400
+	0    1    1    0
+$EndComp
 $EndSCHEMATC
