File: End-Effector_Electronics/End-Effector_Electronics.sch (KiCad schematic (older format))
At the start: 33 parts, among them J1 Raspberry_Pi_2_3, J10 SW_Push_Open, J11 SW_Push_Open, J2 LynxServo, J3 LynxServo, J4 QWIIC_Generic_Conn, J5 Conn_02x05_Odd_Even, J6 AH1815-P-B, J7 AH1815-P-B, J8 AH1815-P-B, J9 SW_Push_Open, Q1 Q_PMOS_GSD, Q2 DMMT3906, Q3 Q_NMOS_GSD, U1 CAT24C32, U2 TDK_I3A4W008A033V

Commit message: Swapped a few components
Parts:
- removed J6, J7, J8: AH1815-P-B, Connector_JST:JST_PH_B3B-PH-K_1x03_P2.00mm_Vertical, symbol Project_Library:AH1815-P-B
- added D2: LED, Connector_JST:JST_PH_B2B-PH-K_1x02_P2.00mm_Vertical, symbol Device:LED
- added LD1: Laserdiode_1C2A, Connector_JST:JST_PH_B2B-PH-K_1x02_P2.00mm_Vertical, symbol Device:Laserdiode_1C2A
- added Q4, Q5: Q_NMOS_GSD, Package_TO_SOT_SMD:SOT-23, symbol Device:Q_NMOS_GSD
- added R10, R11: 100k, Resistor_SMD:R_0603_1608Metric, symbol Device:R_Small
- J1: Digikey Part Num 1528-1785-ND -> (none)
Connections:
- net +12V: now also D2.2 (A)
- net +5V: now also LD1.2 (A)
- net GND: now also Q4.2 (S), Q5.2 (S), R10.2, R11.2
- net Hall1 renamed Laser
- net Laser: now also Q4.1 (G), R10.1
- net Hall2 renamed LED
- net LED: now also Q5.1 (G), R11.1
- net Hall3: no longer names the net of J1.15 (GPIO22)
- new net: LD1.1 (K), Q4.3 (D)
- new net: D2.1 (K), Q5.3 (D)
Changed lines of the file:
@@
 F 2 "Connector_PinSocket_2.54mm:PinSocket_2x20_P2.54mm_Vertical_SMD" H 2150 2600 50  0001 C CNN
 F 3 "https://www.raspberrypi.org/documentation/hardware/raspberrypi/schematics/rpi_SCH_3bplus_1p0_reduced.pdf" H 2150 2600 50  0001 C CNN
-F 4 "1528-1785-ND" H 2150 2600 50  0001 C CNN "Digikey Part Num"
+F 4 "" H 2150 2600 50  0001 C CNN "Digikey Part Num"
 	1    2150 2600
 	1    0    0    -1
@@
 Text Label 1000 2100 2    50   ~ 0
 Limit_SW1
-$Comp
-L Project_Library:AH1815-P-B J6
-U 1 1 61A379AF
-P 7000 2800
-F 0 "J6" H 6770 2846 50  0000 R CNN
-F 1 "AH1815-P-B" H 6770 2755 50  0000 R CNN
-F 2 "Connector_JST:JST_PH_B3B-PH-K_1x03_P2.00mm_Vertical" H 7000 2800 50  0001 C CNN
-F 3 "https://www.diodes.com/assets/Datasheets/AH1806.pdf" H 7000 2800 50  0001 C CNN
-	1    7000 2800
-	1    0    0    -1
-$EndComp
-Text Label 7300 2800 0    50   ~ 0
-Hall1
-$Comp
-L power:+3.3V #PWR030
-U 1 1 61A3AC33
-P 7000 2400
-F 0 "#PWR030" H 7000 2250 50  0001 C CNN
-F 1 "+3.3V" H 7015 2573 50  0000 C CNN
-F 2 "" H 7000 2400 50  0001 C CNN
-F 3 "" H 7000 2400 50  0001 C CNN
-	1    7000 2400
-	1    0    0    -1
-$EndComp
-$Comp
-L power:GND #PWR031
-U 1 1 61A3B102
-P 7000 3200
-F 0 "#PWR031" H 7000 2950 50  0001 C CNN
-F 1 "GND" H 7005 3027 50  0000 C CNN
-F 2 "" H 7000 3200 50  0001 C CNN
-F 3 "" H 7000 3200 50  0001 C CNN
-	1    7000 3200
-	1    0    0    -1
-$EndComp
-$Comp
-L Project_Library:AH1815-P-B J7
-U 1 1 61A3B43B
-P 7000 4150
-F 0 "J7" H 6770 4196 50  0000 R CNN
-F 1 "AH1815-P-B" H 6770 4105 50  0000 R CNN
-F 2 "Connector_JST:JST_PH_B3B-PH-K_1x03_P2.00mm_Vertical" H 7000 4150 50  0001 C CNN
-F 3 "https://www.diodes.com/assets/Datasheets/AH1806.pdf" H 7000 4150 50  0001 C CNN
-	1    7000 4150
-	1    0    0    -1
-$EndComp
-Text Label 7300 4150 0    50   ~ 0
-Hall2
-$Comp
-L power:+3.3V #PWR032
-U 1 1 61A3B950
-P 7000 3750
-F 0 "#PWR032" H 7000 3600 50  0001 C CNN
-F 1 "+3.3V" H 7015 3923 50  0000 C CNN
-F 2 "" H 7000 3750 50  0001 C CNN
-F 3 "" H 7000 3750 50  0001 C CNN
-	1    7000 3750
-	1    0    0    -1
-$EndComp
-$Comp
-L power:GND #PWR033
-U 1 1 61A3B95A
-P 7000 4550
-F 0 "#PWR033" H 7000 4300 50  0001 C CNN
-F 1 "GND" H 7005 4377 50  0000 C CNN
-F 2 "" H 7000 4550 50  0001 C CNN
-F 3 "" H 7000 4550 50  0001 C CNN
-	1    7000 4550
-	1    0    0    -1
-$EndComp
-$Comp
-L Project_Library:AH1815-P-B J8
-U 1 1 61A41319
-P 7000 5500
-F 0 "J8" H 6770 5546 50  0000 R CNN
-F 1 "AH1815-P-B" H 6770 5455 50  0000 R CNN
-F 2 "Connector_JST:JST_PH_B3B-PH-K_1x03_P2.00mm_Vertical" H 7000 5500 50  0001 C CNN
-F 3 "https://www.diodes.com/assets/Datasheets/AH1806.pdf" H 7000 5500 50  0001 C CNN
-	1    7000 5500
-	1    0    0    -1
-$EndComp
-Text Label 7300 5500 0    50   ~ 0
-Hall3
-$Comp
-L power:+3.3V #PWR034
-U 1 1 61A4185E
-P 7000 5100
-F 0 "#PWR034" H 7000 4950 50  0001 C CNN
-F 1 "+3.3V" H 7015 5273 50  0000 C CNN
-F 2 "" H 7000 5100 50  0001 C CNN
-F 3 "" H 7000 5100 50  0001 C CNN
-	1    7000 5100
-	1    0    0    -1
-$EndComp
-$Comp
-L power:GND #PWR035
-U 1 1 61A41868
-P 7000 5900
-F 0 "#PWR035" H 7000 5650 50  0001 C CNN
-F 1 "GND" H 7005 5727 50  0000 C CNN
-F 2 "" H 7000 5900 50  0001 C CNN
-F 3 "" H 7000 5900 50  0001 C CNN
-	1    7000 5900
-	1    0    0    -1
-$EndComp
-Text Label 1000 2800 2    50   ~ 0
-Hall3
 Wire Wire Line
 	1000 2800 1350 2800
@@
 Wire Wire Line
 	1350 2900 1000 2900
+$Comp
+L Device:Laserdiode_1C2A LD1
+U 1 1 619B7CC5
+P 7650 2400
+F 0 "LD1" V 7646 2312 50  0000 R CNN
+F 1 "Laserdiode_1C2A" V 7555 2312 50  0000 R CNN
+F 2 "Connector_JST:JST_PH_B2B-PH-K_1x02_P2.00mm_Vertical" H 7550 2375 50  0001 C CNN
+F 3 "~" H 7680 2200 50  0001 C CNN
+F 4 "1528-1391-ND" H 7650 2400 50  0001 C CNN "Digikey Part Num"
+	1    7650 2400
+	0    -1   -1   0
+$EndComp
+$Comp
+L power:+5V #PWR030
+U 1 1 619B9E92
+P 7650 2100
+F 0 "#PWR030" H 7650 1950 50  0001 C CNN
+F 1 "+5V" H 7665 2273 50  0000 C CNN
+F 2 "" H 7650 2100 50  0001 C CNN
+F 3 "" H 7650 2100 50  0001 C CNN
+	1    7650 2100
+	1    0    0    -1
+$EndComp
+Wire Wire Line
+	7650 2100 7650 2200
+$Comp
+L Device:Q_NMOS_GSD Q4
+U 1 1 619C00A8
+P 7550 3000
+F 0 "Q4" H 7756 3046 50  0000 L CNN
+F 1 "Q_NMOS_GSD" H 7756 2955 50  0000 L CNN
+F 2 "Package_TO_SOT_SMD:SOT-23" H 7750 3100 50  0001 C CNN
+F 3 "~" H 7550 3000 50  0001 C CNN
+F 4 "DMN2041L-7DICT-ND" H 7550 3000 50  0001 C CNN "Digikey Part Num"
+	1    7550 3000
+	1    0    0    -1
+$EndComp
+Wire Wire Line
+	7650 2800 7650 2700
+$Comp
+L power:GND #PWR031
+U 1 1 619C6751
+P 7650 3300
+F 0 "#PWR031" H 7650 3050 50  0001 C CNN
+F 1 "GND" H 7655 3127 50  0000 C CNN
+F 2 "" H 7650 3300 50  0001 C CNN
+F 3 "" H 7650 3300 50  0001 C CNN
+	1    7650 3300
+	1    0    0    -1
+$EndComp
+Wire Wire Line
+	7650 3300 7650 3200
+$Comp
+L Device:R_Small R10
+U 1 1 619CCF73
+P 7200 3100
+F 0 "R10" H 7259 3146 50  0000 L CNN
+F 1 "100k" H 7259 3055 50  0000 L CNN
+F 2 "Resistor_SMD:R_0603_1608Metric" H 7200 3100 50  0001 C CNN
+F 3 "~" H 7200 3100 50  0001 C CNN
+F 4 "311-100KHRCT-ND" H 7200 3100 50  0001 C CNN "Digikey Part Num"
+	1    7200 3100
+	1    0    0    -1
+$EndComp
+Wire Wire Line
+	7350 3000 7200 3000
+Wire Wire Line
+	7200 3200 7650 3200
+Connection ~ 7650 3200
+Wire Wire Line
+	7200 3000 6900 3000
+Connection ~ 7200 3000
+Text Label 6900 3000 0    50   ~ 0
+Laser
+Text Label 1000 3000 2    50   ~ 0
+Laser
+$Comp
+L Device:Q_NMOS_GSD Q5
+U 1 1 619E21EF
+P 7550 4800
+F 0 "Q5" H 7756 4846 50  0000 L CNN
+F 1 "Q_NMOS_GSD" H 7756 4755 50  0000 L CNN
+F 2 "Package_TO_SOT_SMD:SOT-23" H 7750 4900 50  0001 C CNN
+F 3 "~" H 7550 4800 50  0001 C CNN
+F 4 "DMN2041L-7DICT-ND" H 7550 4800 50  0001 C CNN "Digikey Part Num"
+	1    7550 4800
+	1    0    0    -1
+$EndComp
+$Comp
+L power:GND #PWR033
+U 1 1 619E21FA
+P 7650 5100
+F 0 "#PWR033" H 7650 4850 50  0001 C CNN
+F 1 "GND" H 7655 4927 50  0000 C CNN
+F 2 "" H 7650 5100 50  0001 C CNN
+F 3 "" H 7650 5100 50  0001 C CNN
+	1    7650 5100
+	1    0    0    -1
+$EndComp
+Wire Wire Line
+	7650 5100 7650 5000
+$Comp
+L Device:R_Small R11
+U 1 1 619E2206
+P 7200 4900
+F 0 "R11" H 7259 4946 50  0000 L CNN
+F 1 "100k" H 7259 4855 50  0000 L CNN
+F 2 "Resistor_SMD:R_0603_1608Metric" H 7200 4900 50  0001 C CNN
+F 3 "~" H 7200 4900 50  0001 C CNN
+F 4 "311-100KHRCT-ND" H 7200 4900 50  0001 C CNN "Digikey Part Num"
+	1    7200 4900
+	1    0    0    -1
+$EndComp
+Wire Wire Line
+	7350 4800 7200 4800
+Wire Wire Line
+	7200 5000 7650 5000
+Connection ~ 7650 5000
+Wire Wire Line
+	7200 4800 6900 4800
+Connection ~ 7200 4800
+$Comp
+L Device:LED D2
+U 1 1 619F74FA
+P 7650 4250
+F 0 "D2" V 7689 4132 50  0000 R CNN
+F 1 "LED" V 7598 4132 50  0000 R CNN
+F 2 "Connector_JST:JST_PH_B2B-PH-K_1x02_P2.00mm_Vertical" H 7650 4250 50  0001 C CNN
+F 3 "~" H 7650 4250 50  0001 C CNN
+F 4 "1647-1021-1-ND" H 7650 4250 50  0001 C CNN "Digikey Part Num"
+	1    7650 4250
+	0    -1   -1   0
+$EndComp
+Wire Wire Line
+	7650 3900 7650 4100
+Wire Wire Line
+	7650 4400 7650 4600
+$Comp
+L power:+12V #PWR032
+U 1 1 61A069B1
+P 7650 3900
+F 0 "#PWR032" H 7650 3750 50  0001 C CNN
+F 1 "+12V" H 7665 4073 50  0000 C CNN
+F 2 "" H 7650 3900 50  0001 C CNN
+F 3 "" H 7650 3900 50  0001 C CNN
+	1    7650 3900
+	1    0    0    -1
+$EndComp
+Text Label 6900 4800 0    50   ~ 0
+LED
 Text Label 1000 2900 2    50   ~ 0
-Hall2
-Text Label 1000 3000 2    50   ~ 0
-Hall1
+LED
 $EndSCHEMATC

Commit message: Fixed errors
Parts:
- BT1: footprint Connector_AMASS:AMASS_XT30PW-M_1x02_P2.50mm_Horizontal -> Connector_AMASS:AMASS_XT30U-M_1x02_P5.0mm_Vertical
Changed lines of the file:
@@
 F 0 "BT1" H 1378 6996 50  0000 L CNN
 F 1 "XT_Battery_Connector" H 1378 6905 50  0000 L CNN
-F 2 "Connector_AMASS:AMASS_XT30PW-M_1x02_P2.50mm_Horizontal" H 1250 6950 50  0001 C CNN
+F 2 "Connector_AMASS:AMASS_XT30U-M_1x02_P5.0mm_Vertical" H 1250 6950 50  0001 C CNN
 F 3 "" H 1250 6950 50  0001 C CNN
 F 4 "n/a" H 1250 6950 50  0001 C CNN "Digikey Part Num"
