File: End-Effector_Electronics/5v_Supply.sch (KiCad schematic (older format))
At the start: 7 parts, among them U1 LM22676MR-5

Commit message: Started associating components
Parts:
- C1: footprint (none) -> Capacitor_SMD:C_1206_3216Metric; Digikey Part Num (none) -> 1276-6736-1-ND
- C2: footprint (none) -> Capacitor_SMD:C_0805_2012Metric; Digikey Part Num (none) -> 490-10667-1-ND
- C3: footprint (none) -> Capacitor_SMD:C_0603_1608Metric; Digikey Part Num (none) -> 490-4781-1-ND
- C4: footprint (none) -> Capacitor_SMD:C_1206_3216Metric; Digikey Part Num (none) -> 490-12438-1-ND
Changed lines of the file:
@@
 F 0 "C3" H 5908 3854 50  0000 R CNN
 F 1 "10n" H 5908 3945 50  0000 R CNN
-F 2 "" H 6000 3900 50  0001 C CNN
+F 2 "Capacitor_SMD:C_0603_1608Metric" H 6000 3900 50  0001 C CNN
 F 3 "~" H 6000 3900 50  0001 C CNN
+F 4 "490-4781-1-ND" H 6000 3900 50  0001 C CNN "Digikey Part Num"
 	1    6000 3900
 	-1   0    0    1
@@
 F 0 "C2" H 4742 4146 50  0000 L CNN
 F 1 "1u" H 4742 4055 50  0000 L CNN
-F 2 "" H 4650 4100 50  0001 C CNN
+F 2 "Capacitor_SMD:C_0805_2012Metric" H 4650 4100 50  0001 C CNN
 F 3 "~" H 4650 4100 50  0001 C CNN
+F 4 "490-10667-1-ND" H 4650 4100 50  0001 C CNN "Digikey Part Num"
 	1    4650 4100
 	1    0    0    -1
@@
 F 0 "C1" H 4341 4146 50  0000 L CNN
 F 1 "10u" H 4341 4055 50  0000 L CNN
-F 2 "" H 4250 4100 50  0001 C CNN
+F 2 "Capacitor_SMD:C_1206_3216Metric" H 4250 4100 50  0001 C CNN
 F 3 "~" H 4250 4100 50  0001 C CNN
+F 4 "1276-6736-1-ND" H 4250 4100 50  0001 C CNN "Digikey Part Num"
 	1    4250 4100
 	1    0    0    -1
@@
 F 0 "C4" H 7191 4146 50  0000 L CNN
 F 1 "47u" H 7191 4055 50  0000 L CNN
-F 2 "" H 7100 4100 50  0001 C CNN
+F 2 "Capacitor_SMD:C_1206_3216Metric" H 7100 4100 50  0001 C CNN
 F 3 "~" H 7100 4100 50  0001 C CNN
+F 4 "490-12438-1-ND" H 7100 4100 50  0001 C CNN "Digikey Part Num"
 	1    7100 4100
 	1    0    0    -1

Commit message: Worked on finding components
Parts:
- removed C1: 10u, Capacitor_SMD:C_1206_3216Metric, symbol Device:CP1_Small
- removed C4: 47u, Capacitor_SMD:C_1206_3216Metric, symbol Device:CP1_Small
- added C10, C9: 47u, Capacitor_SMD:C_1210_3225Metric, symbol Device:C_Small
- added C4, C5, C6: 10u, Capacitor_SMD:C_1210_3225Metric, symbol Device:C_Small
- C8: renamed from C3; Digikey Part Num 490-4781-1-ND -> 311-1085-1-ND
- D1: footprint (none) -> Diode_SMD:D_PowerDI-5; Digikey Part Num (none) -> PDS560DICT-ND
- L1: footprint (none) -> Inductor_SMD:L_Wuerth_HCI-1050; Digikey Part Num (none) -> 732-4180-1-ND
- renumbered C2 to C7, U1 to U3
Connections:
- net Vin+: now also C4.1, C5.1, C6.1
- net Vin-: now also C10.2, C4.2, C5.2, C6.2, C9.2
- net Vout+: now also C10.1, C9.1
Changed lines of the file:
@@
 Vout+
 $Comp
-L Regulator_Switching:LM22676MR-5 U1
+L Regulator_Switching:LM22676MR-5 U3
 U 1 1 617DB04C
 P 5450 4000
-F 0 "U1" H 5450 4467 50  0000 C CNN
+F 0 "U3" H 5450 4467 50  0000 C CNN
 F 1 "LM22676MR-5" H 5450 4376 50  0000 C CNN
 F 2 "Package_SO:TI_SO-PowerPAD-8" H 5450 4450 50  0001 C CNN
@@
 Connection ~ 5550 4850
 $Comp
-L Device:C_Small C3
+L Device:C_Small C8
 U 1 1 617DBA3C
 P 6000 3900
-F 0 "C3" H 5908 3854 50  0000 R CNN
+F 0 "C8" H 5908 3854 50  0000 R CNN
 F 1 "10n" H 5908 3945 50  0000 R CNN
 F 2 "Capacitor_SMD:C_0603_1608Metric" H 6000 3900 50  0001 C CNN
 F 3 "~" H 6000 3900 50  0001 C CNN
-F 4 "490-4781-1-ND" H 6000 3900 50  0001 C CNN "Digikey Part Num"
+F 4 "311-1085-1-ND" H 6000 3900 50  0001 C CNN "Digikey Part Num"
 	1    6000 3900
 	-1   0    0    1
@@
 F 0 "L1" V 6790 3800 50  0000 C CNN
 F 1 "18u" V 6699 3800 50  0000 C CNN
-F 2 "" H 6600 3800 50  0001 C CNN
+F 2 "Inductor_SMD:L_Wuerth_HCI-1050" H 6600 3800 50  0001 C CNN
 F 3 "~" H 6600 3800 50  0001 C CNN
+F 4 "732-4180-1-ND" H 6600 3800 50  0001 C CNN "Digikey Part Num"
 	1    6600 3800
 	0    -1   -1   0
@@
 F 0 "D1" V 6304 4080 50  0000 L CNN
 F 1 "D_Schottky" V 6395 4080 50  0000 L CNN
-F 2 "" H 6350 4000 50  0001 C CNN
+F 2 "Diode_SMD:D_PowerDI-5" H 6350 4000 50  0001 C CNN
 F 3 "~" H 6350 4000 50  0001 C CNN
+F 4 "PDS560DICT-ND" H 6350 4000 50  0001 C CNN "Digikey Part Num"
 	1    6350 4000
 	0    1    1    0
 $EndComp
 $Comp
-L Device:C_Small C2
+L Device:C_Small C7
 U 1 1 617DCE06
 P 4650 4100
-F 0 "C2" H 4742 4146 50  0000 L CNN
+F 0 "C7" H 4742 4146 50  0000 L CNN
 F 1 "1u" H 4742 4055 50  0000 L CNN
 F 2 "Capacitor_SMD:C_0805_2012Metric" H 4650 4100 50  0001 C CNN
@@
 	1    0    0    -1
 $EndComp
-$Comp
-L Device:CP1_Small C1
-U 1 1 617DD0A0
-P 4250 4100
-F 0 "C1" H 4341 4146 50  0000 L CNN
-F 1 "10u" H 4341 4055 50  0000 L CNN
-F 2 "Capacitor_SMD:C_1206_3216Metric" H 4250 4100 50  0001 C CNN
-F 3 "~" H 4250 4100 50  0001 C CNN
-F 4 "1276-6736-1-ND" H 4250 4100 50  0001 C CNN "Digikey Part Num"
-	1    4250 4100
-	1    0    0    -1
-$EndComp
 Wire Wire Line
 	4150 3800 4250 3800
@@
 	6900 3800 6750 3800
 Wire Wire Line
-	7100 4200 7100 4850
-Wire Wire Line
 	7100 4000 7100 3800
-$Comp
-L Device:CP1_Small C4
-U 1 1 617DBFA8
-P 7100 4100
-F 0 "C4" H 7191 4146 50  0000 L CNN
-F 1 "47u" H 7191 4055 50  0000 L CNN
-F 2 "Capacitor_SMD:C_1206_3216Metric" H 7100 4100 50  0001 C CNN
-F 3 "~" H 7100 4100 50  0001 C CNN
-F 4 "490-12438-1-ND" H 7100 4100 50  0001 C CNN "Digikey Part Num"
-	1    7100 4100
-	1    0    0    -1
-$EndComp
 Connection ~ 7100 3800
 Connection ~ 7100 4850
@@
 Wire Wire Line
 	6900 3800 7100 3800
+$Comp
+L Device:C_Small C6
+U 1 1 619850EE
+P 4250 4100
+F 0 "C6" H 4342 4146 50  0000 L CNN
+F 1 "10u" H 4342 4055 50  0000 L CNN
+F 2 "Capacitor_SMD:C_1210_3225Metric" H 4250 4100 50  0001 C CNN
+F 3 "~" H 4250 4100 50  0001 C CNN
+F 4 "445-181658-1-ND" H 4250 4100 50  0001 C CNN "Digikey Part Num"
+	1    4250 4100
+	1    0    0    -1
+$EndComp
+$Comp
+L Device:C_Small C5
+U 1 1 6198621A
+P 3950 4100
+F 0 "C5" H 4042 4146 50  0000 L CNN
+F 1 "10u" H 4042 4055 50  0000 L CNN
+F 2 "Capacitor_SMD:C_1210_3225Metric" H 3950 4100 50  0001 C CNN
+F 3 "~" H 3950 4100 50  0001 C CNN
+F 4 "445-181658-1-ND" H 3950 4100 50  0001 C CNN "Digikey Part Num"
+	1    3950 4100
+	1    0    0    -1
+$EndComp
+$Comp
+L Device:C_Small C4
+U 1 1 6198656B
+P 3700 4100
+F 0 "C4" H 3792 4146 50  0000 L CNN
+F 1 "10u" H 3792 4055 50  0000 L CNN
+F 2 "Capacitor_SMD:C_1210_3225Metric" H 3700 4100 50  0001 C CNN
+F 3 "~" H 3700 4100 50  0001 C CNN
+F 4 "445-181658-1-ND" H 3700 4100 50  0001 C CNN "Digikey Part Num"
+	1    3700 4100
+	1    0    0    -1
+$EndComp
+Wire Wire Line
+	3700 4000 3950 4000
+Connection ~ 4250 4000
+Connection ~ 3950 4000
+Wire Wire Line
+	3950 4000 4250 4000
+Wire Wire Line
+	4250 4200 3950 4200
+Connection ~ 4250 4200
+Connection ~ 3950 4200
+Wire Wire Line
+	3950 4200 3700 4200
+Wire Wire Line
+	7100 4200 7100 4850
+$Comp
+L Device:C_Small C9
+U 1 1 619877D0
+P 7100 4100
+F 0 "C9" H 7192 4146 50  0000 L CNN
+F 1 "47u" H 7192 4055 50  0000 L CNN
+F 2 "Capacitor_SMD:C_1210_3225Metric" H 7100 4100 50  0001 C CNN
+F 3 "~" H 7100 4100 50  0001 C CNN
+F 4 "732-7382-1-ND" H 7100 4100 50  0001 C CNN "Digikey Part Num"
+	1    7100 4100
+	1    0    0    -1
+$EndComp
+$Comp
+L Device:C_Small C10
+U 1 1 61987CA6
+P 7400 4100
+F 0 "C10" H 7492 4146 50  0000 L CNN
+F 1 "47u" H 7492 4055 50  0000 L CNN
+F 2 "Capacitor_SMD:C_1210_3225Metric" H 7400 4100 50  0001 C CNN
+F 3 "~" H 7400 4100 50  0001 C CNN
+F 4 "732-7382-1-ND" H 7400 4100 50  0001 C CNN "Digikey Part Num"
+	1    7400 4100
+	1    0    0    -1
+$EndComp
+Wire Wire Line
+	7100 4200 7400 4200
+Connection ~ 7100 4200
+Wire Wire Line
+	7400 4000 7100 4000
+Connection ~ 7100 4000
 $EndSCHEMATC

Commit message: More component part selection
Parts:
- U3: Digikey Part Num (none) -> LM22676MR-5.0/NOPB-ND
Changed lines of the file:
@@
 F 2 "Package_SO:TI_SO-PowerPAD-8" H 5450 4450 50  0001 C CNN
 F 3 "http://www.ti.com/lit/ds/symlink/lm22676.pdf" H 5500 4000 50  0001 C CNN
+F 4 "LM22676MR-5.0/NOPB-ND" H 5450 4000 50  0001 C CNN "Digikey Part Num"
 	1    5450 4000
 	1    0    0    -1
